File: PCB/WindTurbineController.kicad_pcb (KiCad board)
At the start: 2 copper layers, 19 parts, among them Q1 2N7000, Q2 2N7000, Q3 2N7000, Q4 2N7000

Commit message: PCB implemented.
Parts:
- added D1: 1N4001, Diode_THT:D_DO-41_SOD81_P2.54mm_Vertical_AnodeUp, F.Cu at (72.5, 73.2)
- added J1: Conn_01x06_Male, Connector_PinHeader_2.54mm:PinHeader_1x06_P2.54mm_Vertical, F.Cu at (36.2, 66.4)
- added J2: Screw_Terminal_01x03, TerminalBlock:TerminalBlock_bornier-3_P5.08mm, F.Cu at (91.8, 78.2)
- added J3: Screw_Terminal_01x02, TerminalBlock:TerminalBlock_bornier-2_P5.08mm, F.Cu at (95.2, 48.9)
- added J4: Screw_Terminal_01x02, TerminalBlock:TerminalBlock_bornier-2_P5.08mm, F.Cu at (91.4, 65.5)
- added K1: SANYOU_SRD_Form_C, Relay_THT:Relay_SPDT_SANYOU_SRD_Series_Form_C, F.Cu at (68.5, 83.2)
- added Q5: BC337, Package_TO_SOT_THT:TO-92_Inline, F.Cu at (65.0, 88.6)
- added R15: 4k7, Resistor_THT:R_Axial_DIN0207_L6.3mm_D2.5mm_P2.54mm_Vertical, F.Cu at (64.0, 76.8)
- added R16: 470, Resistor_THT:R_Axial_DIN0207_L6.3mm_D2.5mm_P2.54mm_Vertical, F.Cu at (64.0, 84.8)
- added R17: 1k, Resistor_THT:R_Axial_DIN0207_L6.3mm_D2.5mm_P2.54mm_Vertical, F.Cu at (92.2, 59.6)
- added R18: 10k, Resistor_THT:R_Axial_DIN0207_L6.3mm_D2.5mm_P2.54mm_Vertical, F.Cu at (83.0, 56.8)
- added R19: 2k, Resistor_THT:R_Axial_DIN0207_L6.3mm_D2.5mm_P2.54mm_Vertical, F.Cu at (83.6, 68.8)
- added R20: 1k, Resistor_THT:R_Axial_DIN0207_L6.3mm_D2.5mm_P2.54mm_Vertical, F.Cu at (85.6, 72.0)
- added SW1: SW_Push, Arduino_Library:SW_Push_Unknown, F.Cu at (49.2, 55.2)
- added SW2: SW_Push, Arduino_Library:SW_Push_Unknown, F.Cu at (53.6, 83.4)
- added SW3: SW_Push, Arduino_Library:SW_Push_Unknown, F.Cu at (51.6, 69.6)
- added U1: PC817, Package_DIP:DIP-4_W7.62mm, F.Cu at (86.7, 56.0)
- R1, R2, R3, R4, R5, R6, R7, R8: footprint Resistor_THT:R_Axial_DIN0207_L6.3mm_D2.5mm_P7.62mm_Horizontal -> Resistor_THT:R_Axial_DIN0207_L6.3mm_D2.5mm_P2.54mm_Vertical
- R10, R12, R14: value R -> 220; footprint Resistor_THT:R_Axial_DIN0204_L3.6mm_D1.6mm_P5.08mm_Horizontal -> Resistor_THT:R_Axial_DIN0207_L6.3mm_D2.5mm_P2.54mm_Vertical
- R11, R13, R9: value R -> 12k; footprint Resistor_THT:R_Axial_DIN0204_L3.6mm_D1.6mm_P5.08mm_Horizontal -> Resistor_THT:R_Axial_DIN0207_L6.3mm_D2.5mm_P2.54mm_Vertical
- moved Q2 210.1 mm to (70.5, 61.6)
- moved R3 198.1 mm to (70.3, 67.3), turned to 90 degrees
- moved R4 195.8 mm to (73.3, 67.3), turned to 90 degrees
- moved R12 167.5 mm to (43.0, 75.0), turned to 90 degrees
- moved R11 164.2 mm to (43.0, 78.4), turned to -90 degrees
- moved Q4 149.5 mm to (77.4, 50.9), turned to 90 degrees
- moved R7 132.7 mm to (83.1, 51.1), turned to 180 degrees
- moved R8 132.4 mm to (83.1, 48.1), turned to 180 degrees
- moved R14 127.1 mm to (63.6, 70.1), turned to -90 degrees
- moved R13 127.1 mm to (63.6, 67.0), turned to 90 degrees
- moved Q1 84.9 mm to (62.8, 50.5)
- moved R9 76.0 mm to (58.2, 53.4), turned to 90 degrees
- moved R10 75.9 mm to (58.2, 56.6), turned to -90 degrees
- moved R6 75.3 mm to (73.0, 55.9), turned to 90 degrees
- moved R1 74.9 mm to (62.6, 56.1), turned to 90 degrees
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Connections:
- XA1 pad D0: unconnected-(XA1-PadD0) -> Net-(R16-Pad2)
- XA1 pad D11: unconnected-(XA1-PadD11) -> /level_translator_2/5V_IO
- XA1 pad D13: unconnected-(XA1-PadD13) -> /level_translator_1/5V_IO
- XA1 pad D2: /btn3/btn_in -> Net-(R18-Pad1)
- XA1 pad D3: /btn2/btn_in -> Net-(R19-Pad1)
- XA1 pad D4: /btn1/btn_in -> unconnected-(XA1-PadD4)
- XA1 pad D5: unconnected-(XA1-PadD5) -> /btn3/btn_in
- XA1 pad D6: unconnected-(XA1-PadD6) -> /btn2/btn_in
- XA1 pad D7: unconnected-(XA1-PadD7) -> /btn1/btn_in
- XA1 pad GND2: unconnected-(XA1-PadGND2) -> GND
- XA1 pad GND3: unconnected-(XA1-PadGND3) -> GND
- XA1 pad MOSI: /level_translator_2/5V_IO -> unconnected-(XA1-PadMOSI)
- XA1 pad SCK: /level_translator_1/5V_IO -> unconnected-(XA1-PadSCK)
Routing:
- net +3.3V: track 0.00 -> 145.6 mm, vias 0 -> 2
- net +5V: track 0.00 -> 144.3 mm, vias 0 -> 7
- net /btn2/btn_in: track 0.00 -> 66.1 mm, vias 0 -> 4
- net Net-(R16-Pad2): track 0.00 -> 63.6 mm, vias 0 -> 1
- net /level_translator_4/3V_IO: track 0.00 -> 60.1 mm, vias 0 -> 4
- net /level_translator_3/3V_IO: track 0.00 -> 49.5 mm, vias 0 -> 2
- net /btn3/btn_in: track 0.00 -> 46.3 mm
- net /level_translator_1/3V_IO: track 0.00 -> 45.6 mm, vias 0 -> 2
- net /level_translator_2/3V_IO: track 0.00 -> 42.0 mm, vias 0 -> 2
- net /btn1/btn_in: track 0.00 -> 39.4 mm, vias 0 -> 2
- net Net-(R19-Pad1): track 0.00 -> 39.1 mm, vias 0 -> 1
- net Net-(R13-Pad2): track 0.00 -> 35.5 mm, vias 0 -> 1
- net Net-(R10-Pad1): track 0.00 -> 31.6 mm, vias 0 -> 1
- net Net-(R11-Pad2): track 0.00 -> 28.5 mm
- net Net-(J2-Pad3): track 0.00 -> 25.4 mm
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- added copper zone on B.Cu, net GND
- added copper zone on F.Cu, net GND
Other:
- board outline added: 70.4 x 55.6 mm
- board text added: "NC"
- board text added: "NO"
- board text added: "OPTO"
- board text added: "V.D."
