File: PCB/WindTurbineController.kicad_sch (KiCad schematic)
At the start: 8 parts, among them J1 Conn_01x06_Male

Commit message: PCB implemented.
Parts:
- added J2: Screw_Terminal_01x03, TerminalBlock:TerminalBlock_bornier-3_P5.08mm, symbol Connector:Screw_Terminal_01x03
- added J3, J4: Screw_Terminal_01x02, TerminalBlock:TerminalBlock_bornier-2_P5.08mm, symbol Connector:Screw_Terminal_01x02
- added R17, R20: 1k, Resistor_THT:R_Axial_DIN0207_L6.3mm_D2.5mm_P2.54mm_Vertical, symbol Device:R
- added R18: 10k, Resistor_THT:R_Axial_DIN0207_L6.3mm_D2.5mm_P2.54mm_Vertical, symbol Device:R
- added R19: 2k, Resistor_THT:R_Axial_DIN0207_L6.3mm_D2.5mm_P2.54mm_Vertical, symbol Device:R
- D1: renamed from D?; footprint Diode_THT:D_DO-41_SOD81_P10.16mm_Horizontal -> Diode_THT:D_DO-41_SOD81_P2.54mm_Vertical_AnodeUp
- J1: footprint (none) -> Connector_PinHeader_2.54mm:PinHeader_1x06_P2.54mm_Vertical
- R15, R16: renamed from R?; footprint (none) -> Resistor_THT:R_Axial_DIN0207_L6.3mm_D2.5mm_P2.54mm_Vertical
- gave numbers to parts that had none: 3
Connections:
- net +5V: now also U1.4
- net GND: now also XA1.GND2 (GND), XA1.GND3 (GND), J4.2 (Pin_2), R18.2, R20.1
- net at K1.1: now also J2.3 (Pin_3)
- net at K1.3: now also J2.2 (Pin_2)
- net at K1.4: now also J2.1 (Pin_1)
- net at U1.1: now also R17.2
- net at U1.2: now also J3.1 (Pin_1)
- net at U1.3: now also XA1.D2 (D2_INT0), R18.1
- net at XA1.D3 (D3_INT1): now also R19.1, R20.2
- new net: J4.1 (Pin_1), R19.2
- new net: J3.2 (Pin_2), R17.1
- no-connect marks 0 -> 22
Other:
- moved on the sheet: U1
