File: PCB/btn1.kicad_sch (KiCad schematic)
At the start: 3 parts, among them SW3 SW_Push

Commit message: PCB implemented.
Parts:
- R13: value R -> 12k; footprint Resistor_THT:R_Axial_DIN0204_L3.6mm_D1.6mm_P5.08mm_Horizontal -> Resistor_THT:R_Axial_DIN0207_L6.3mm_D2.5mm_P2.54mm_Vertical
- R14: value R -> 220; footprint Resistor_THT:R_Axial_DIN0204_L3.6mm_D1.6mm_P5.08mm_Horizontal -> Resistor_THT:R_Axial_DIN0207_L6.3mm_D2.5mm_P2.54mm_Vertical
- SW3: footprint (none) -> Arduino_Library:SW_Push_Unknown
Changed lines of the file:
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@@
     (property "Reference" "SW3" (id 0) (at 146.05 88.9 0))
     (property "Value" "SW_Push" (id 1) (at 146.05 91.44 0))
-    (property "Footprint" "" (id 2) (at 146.05 91.44 0)
+    (property "Footprint" "Arduino_Library:SW_Push_Unknown" (id 2) (at 146.05 91.44 0)
       (effects (font (size 1.27 1.27)) hide)
     )
@@
   (symbol (lib_id "Device:R") (at 137.16 91.44 0) (unit 1)
     (in_bom yes) (on_board yes) (fields_autoplaced)
-    (property "Reference" "R13" (id 0) (at 139.7 90.1699 0)
+    (property "Reference" "R13" (id 0) (at 138.938 90.6053 0)
       (effects (font (size 1.27 1.27)) (justify left))
     )
-    (property "Value" "R" (id 1) (at 139.7 92.7099 0)
+    (property "Value" "12k" (id 1) (at 138.938 93.1422 0)
       (effects (font (size 1.27 1.27)) (justify left))
     )
-    (property "Footprint" "Resistor_THT:R_Axial_DIN0204_L3.6mm_D1.6mm_P5.08mm_Horizontal" (id 2) (at 135.382 91.44 90)
+    (property "Footprint" "Resistor_THT:R_Axial_DIN0207_L6.3mm_D2.5mm_P2.54mm_Vertical" (id 2) (at 135.382 91.44 90)
       (effects (font (size 1.27 1.27)) hide)
     )
@@
   (symbol (lib_id "Device:R") (at 137.16 101.6 0) (unit 1)
     (in_bom yes) (on_board yes) (fields_autoplaced)
-    (property "Reference" "R14" (id 0) (at 139.7 100.3299 0)
+    (property "Reference" "R14" (id 0) (at 138.938 100.7653 0)
       (effects (font (size 1.27 1.27)) (justify left))
     )
-    (property "Value" "R" (id 1) (at 139.7 102.8699 0)
+    (property "Value" "220" (id 1) (at 138.938 103.3022 0)
       (effects (font (size 1.27 1.27)) (justify left))
     )
-    (property "Footprint" "Resistor_THT:R_Axial_DIN0204_L3.6mm_D1.6mm_P5.08mm_Horizontal" (id 2) (at 135.382 101.6 90)
+    (property "Footprint" "Resistor_THT:R_Axial_DIN0207_L6.3mm_D2.5mm_P2.54mm_Vertical" (id 2) (at 135.382 101.6 90)
       (effects (font (size 1.27 1.27)) hide)
     )
